Commit message: msg

File: robots/sr_hand_bimanual.urdf (robot description, URDF)
Before this commit: robot bimanual_shadowhand_motor, 65 links, 64 joints
Joints:
- joint lh_THJ1: type revolute -> fixed
- joint lh_THJ2: type revolute -> fixed
- joint lh_THJ3: type revolute -> fixed
- joint lh_THJ4: origin xyz=0 0 0 rpy=0 0 0 -> xyz=0 0 0 rpy=0 -1.5708 0; type revolute -> fixed
- joint lh_THJ5: origin xyz=-0.034 -0.00858 0.029 rpy=-0.7853981633974483 0 1.5707963267948966 -> xyz=-0.034 -0.00858 0.029 rpy=-1.5707963267948966 0 1.5707963267948966
- joint rh_THJ1: type revolute -> fixed
- joint rh_THJ2: type revolute -> fixed
- joint rh_THJ3: type revolute -> fixed
- joint rh_THJ4: type revolute -> fixed
- joint rh_THJ5: origin xyz=0.034 -0.00858 0.029 rpy=-0.7853981633974483 0 -1.5707963267948966 -> xyz=0.034 -0.00858 0.029 rpy=0.0 0.0 -1.5707963267948966; type revolute -> fixed
- joint right_hand_to_left_hand: axis (none) -> -1 0 0; limit (none) -> lower=0.2 upper=1 effort=1000 velocity=0.5; origin xyz=-0.4 0.0 0.0 rpy=0.0 0.0 0.0 -> xyz=0.2 -0.45 0.4 rpy=1.5708 0 3.1415; type fixed -> prismatic
- joint world_joint: origin xyz=0.0 0.0 0.0 rpy=0.0 0.0 0.0 -> xyz=0.0 0.0 0.2 rpy=-1.5708 3.1415 0

Commit message: msg

File: robots/sr_hand_bimanual.urdf (robot description, URDF)
Before this commit: robot bimanual_shadowhand_motor, 65 links, 64 joints
Links:
- added link lh_wrist_intermediate
Joints:
- added joint lh_WRJ3: type revolute, parent lh_forearm, child lh_wrist_intermediate, origin xyz=0 -0.010 0.21301 rpy=0 0 0, axis 0 0 1, limit lower=-1.4 upper=1.5708 effort=30 velocity=2.0
- joint lh_THJ1: type fixed -> revolute
- joint lh_THJ2: type fixed -> revolute
- joint lh_THJ3: type fixed -> revolute
- joint lh_THJ4: type fixed -> revolute
- joint lh_WRJ2: origin xyz=0 -0.010 0.21301 rpy=0 0 0 -> xyz=0 0 0 rpy=0 0 0; parent lh_forearm -> lh_wrist_intermediate
- joint right_hand_to_left_hand: origin xyz=0.2 -0.45 0.4 rpy=1.5708 0 3.1415 -> xyz=0 -0.375 0.5 rpy=1.5708 0 3.1415

Commit message: Changed thumb position

File: robots/sr_hand_bimanual.urdf (robot description, URDF)
Before this commit: robot bimanual_shadowhand_motor, 66 links, 65 joints
Joints:
- joint rh_THJ1: origin xyz=0 0 0.032 rpy=0 0 0 -> xyz=0 0 0.032 rpy=0.265 0 0
- joint rh_THJ2: origin xyz=0 0 0 rpy=0 0 0 -> xyz=0 0 0 rpy=0.366 0 0
- joint rh_THJ3: origin xyz=0 0 0.038 rpy=0 0 0 -> xyz=0 0 0.038 rpy=0 0.110 0
- joint rh_THJ4: origin xyz=0 0 0 rpy=0 0 0 -> xyz=0 0 0 rpy=0 0.205 0
- joint rh_THJ5: origin xyz=0.034 -0.00858 0.029 rpy=0.0 0.0 -1.5707963267948966 -> xyz=0.034 -0.00858 0.029 rpy=0.0 0.0 -1.0457963267948966

Commit message: fine-tuned lambdas and added print statements

File: robots/sr_hand_bimanual.urdf (robot description, URDF)
Before this commit: robot bimanual_shadowhand_motor, 66 links, 65 joints
Joints:
- joint right_hand_to_left_hand: origin xyz=0 -0.375 0.5 rpy=1.5708 0 3.1415 -> xyz=0 -0.375 0.500 rpy=1.5708 0 3.1415

Commit message: Change thumb

File: robots/sr_hand_bimanual.urdf (robot description, URDF)
Before this commit: robot bimanual_shadowhand_motor, 66 links, 65 joints
Joints:
- joint rh_THJ5: origin xyz=0.034 -0.00858 0.029 rpy=0.0 0.0 -1.0457963267948966 -> xyz=0.034 -0.00858 0.029 rpy=0.0 0.0 -2

Commit message: Han

File: robots/sr_hand_bimanual.urdf (robot description, URDF)
Before this commit: robot bimanual_shadowhand_motor, 66 links, 65 joints
Joints:
- joint rh_THJ4: origin xyz=0 0 0 rpy=0 0.205 0 -> xyz=0 0 0 rpy=0 -0.205 0
- joint rh_THJ5: origin xyz=0.034 -0.00858 0.029 rpy=0.0 0.0 -2 -> xyz=0.034 -0.00858 0.029 rpy=0.0 0.0 -1.0457963267948966

Commit message: Thumb

File: robots/sr_hand_bimanual.urdf (robot description, URDF)
Before this commit: robot bimanual_shadowhand_motor, 66 links, 65 joints
Joints:
- joint rh_THJ4: origin xyz=0 0 0 rpy=0 -0.205 0 -> xyz=0 0 0 rpy=0 0.4 0

Commit message: Th

File: robots/sr_hand_bimanual.urdf (robot description, URDF)
Before this commit: robot bimanual_shadowhand_motor, 66 links, 65 joints
Joints:
- joint rh_THJ4: origin xyz=0 0 0 rpy=0 0.4 0 -> xyz=0 0 0 rpy=0 0.6 0

Commit message: Th2

File: robots/sr_hand_bimanual.urdf (robot description, URDF)
Before this commit: robot bimanual_shadowhand_motor, 66 links, 65 joints
Joints:
- joint rh_THJ4: origin xyz=0 0 0 rpy=0 0.6 0 -> xyz=0 0 0 rpy=0 0.65 0

Commit message: moved hands a bit

File: robots/sr_hand_bimanual.urdf (robot description, URDF)
Before this commit: robot bimanual_shadowhand_motor, 66 links, 65 joints
Joints:
- joint right_hand_to_left_hand: origin xyz=0 -0.375 0.500 rpy=1.5708 0 3.1415 -> xyz=0 -0.375 0.420 rpy=1.5708 0 3.1415
- joint world_joint: origin xyz=0.0 0.0 0.2 rpy=-1.5708 3.1415 0 -> xyz=0.0 0.0 0.200 rpy=-1.5708 3.1415 0

Commit message: moved hands a bit to make strumming look more natural

File: robots/sr_hand_bimanual.urdf (robot description, URDF)
Before this commit: robot bimanual_shadowhand_motor, 66 links, 65 joints
Joints:
- joint right_hand_to_left_hand: origin xyz=0 -0.375 0.420 rpy=1.5708 0 3.1415 -> xyz=0 -0.455 0.400 rpy=1.5708 0 3.1415
- joint world_joint: origin xyz=0.0 0.0 0.200 rpy=-1.5708 3.1415 0 -> xyz=0.0 0.0 0.280 rpy=-1.5708 3.1415 0
